File: Akashi-12.kicad_sch (KiCad schematic)
At the start: 28 parts, among them J1 USB Type-C receptacle, SW1 SW_MEC_5E, SW2 SW_MEC_5E, U1 RP2040, U2 W25Q32JVSS, U3 NCP1117-3.3_SOT223, Y1 12MHz

Commit message: Place parts on the layout.
Parts:
- added C14, C15: 0.1u, Capacitor_SMD:C_0603_1608Metric_Pad1.08x0.95mm_HandSolder, symbol Device:C
- U1: footprint IC57_RP2040 -> Local:RP2040
Connections:
- net +3V3: now also C14.1, C15.1
- net GND: now also C14.2, C15.2
Other:
- note added: "C7 should be placed closed to pin 44 of U1. C11 should be placed closed to pin 45 of U1."
Changed lines of the file:
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@@
   (junction (at 63.5 175.26) (diameter 0) (color 0 0 0 0)
   )
+  (junction (at 179.07 130.81) (diameter 0) (color 0 0 0 0)
+  )
   (junction (at 254 143.51) (diameter 0) (color 0 0 0 0)
   )
+  (junction (at 179.07 143.51) (diameter 0) (color 0 0 0 0)
+  )
   (junction (at 251.46 46.99) (diameter 0) (color 0 0 0 0)
   )
@@
   (junction (at 213.36 143.51) (diameter 0) (color 0 0 0 0)
   )
+  (junction (at 167.64 143.51) (diameter 0) (color 0 0 0 0)
+  )
   (junction (at 107.95 156.21) (diameter 0) (color 0 0 0 0)
   )
@@
   )
   (junction (at 224.79 130.81) (diameter 0) (color 0 0 0 0)
+  )
+  (junction (at 167.64 130.81) (diameter 0) (color 0 0 0 0)
   )
   (no_connect (at 138.43 85.09))
@@
     (stroke (width 0) (type default) (color 0 0 0 0))
   )
+  (wire (pts (xy 156.21 143.51) (xy 167.64 143.51))
+    (stroke (width 0) (type default) (color 0 0 0 0))
+  )
   (wire (pts (xy 77.47 92.71) (xy 74.93 92.71))
     (stroke (width 0) (type default) (color 0 0 0 0))
@@
     (stroke (width 0) (type default) (color 0 0 0 0))
   )
+  (wire (pts (xy 179.07 143.51) (xy 167.64 143.51))
+    (stroke (width 0) (type default) (color 0 0 0 0))
+  )
   (wire (pts (xy 190.5 130.81) (xy 201.93 130.81))
     (stroke (width 0) (type default) (color 0 0 0 0))
@@
     (stroke (width 0) (type default) (color 0 0 0 0))
   )
+  (wire (pts (xy 167.64 140.97) (xy 167.64 143.51))
+    (stroke (width 0) (type default) (color 0 0 0 0))
+  )
   (wire (pts (xy 265.43 140.97) (xy 265.43 143.51))
     (stroke (width 0) (type default) (color 0 0 0 0))
@@
     (stroke (width 0) (type default) (color 0 0 0 0))
   )
+  (wire (pts (xy 156.21 133.35) (xy 156.21 130.81))
+    (stroke (width 0) (type default) (color 0 0 0 0))
+  )
+  (wire (pts (xy 156.21 130.81) (xy 167.64 130.81))
+    (stroke (width 0) (type default) (color 0 0 0 0))
+  )
   (wire (pts (xy 60.96 90.17) (xy 60.96 95.25))
     (stroke (width 0) (type default) (color 0 0 0 0))
@@
     (stroke (width 0) (type default) (color 0 0 0 0))
   )
+  (wire (pts (xy 167.64 130.81) (xy 179.07 130.81))
+    (stroke (width 0) (type default) (color 0 0 0 0))
+  )
   (wire (pts (xy 151.13 62.23) (xy 153.67 62.23))
     (stroke (width 0) (type default) (color 0 0 0 0))
@@
     (stroke (width 0) (type default) (color 0 0 0 0))
   )
+  (wire (pts (xy 167.64 133.35) (xy 167.64 130.81))
+    (stroke (width 0) (type default) (color 0 0 0 0))
+  )
   (wire (pts (xy 143.51 59.69) (xy 143.51 34.29))
     (stroke (width 0) (type default) (color 0 0 0 0))
@@
     (stroke (width 0) (type default) (color 0 0 0 0))
   )
+  (wire (pts (xy 156.21 140.97) (xy 156.21 143.51))
+    (stroke (width 0) (type default) (color 0 0 0 0))
+  )
   (wire (pts (xy 60.96 95.25) (xy 52.07 95.25))
     (stroke (width 0) (type default) (color 0 0 0 0))
@@
   (wire (pts (xy 151.13 64.77) (xy 151.13 62.23))
     (stroke (width 0) (type default) (color 0 0 0 0))
+  )
+  (text "C7  should be placed closed to pin 44 of U1.\nC11 should be placed closed to pin 45 of U1."
+    (at 181.61 162.56 0)
+    (effects (font (size 2.54 2.54)) (justify left bottom))
   )
   (label "QSPI_SD0" (at 151.13 49.53 0)
@@
       (effects (font (size 1.524 1.524)))
     )
-    (property "Footprint" "IC57_RP2040" (id 2) (at 107.95 33.274 0)
+    (property "Footprint" "Local:RP2040" (id 2) (at 107.95 33.274 0)
       (effects (font (size 1.524 1.524)) hide)
     )
@@
   (symbol (lib_id "power:GND") (at 72.39 123.19 0) (unit 1)
     (in_bom yes) (on_board yes) (fields_autoplaced)
-    (property "Reference" "#PWR?" (id 0) (at 72.39 129.54 0)
+    (property "Reference" "#PWR0103" (id 0) (at 72.39 129.54 0)
       (effects (font (size 1.27 1.27)) hide)
     )
@@
     (pin "2")
   )
+  (symbol (lib_id "Device:C") (at 167.64 137.16 0) (unit 1)
+    (in_bom yes) (on_board yes) (fields_autoplaced)
+    (property "Reference" "C15" (id 0) (at 171.45 135.8899 0)
+      (effects (font (size 1.27 1.27)) (justify left))
+    )
+    (property "Value" "0.1u" (id 1) (at 171.45 138.4299 0)
+      (effects (font (size 1.27 1.27)) (justify left))
+    )
+    (property "Footprint" "Capacitor_SMD:C_0603_1608Metric_Pad1.08x0.95mm_HandSolder" (id 2) (at 168.6052 140.97 0)
+      (effects (font (size 1.27 1.27)) hide)
+    )
+    (property "Datasheet" "~" (id 3) (at 167.64 137.16 0)
+      (effects (font (size 1.27 1.27)) hide)
+    )
+    (pin "1")
+    (pin "2")
+  )
   (symbol (lib_id "Switch:SW_MEC_5E") (at 68.58 115.57 90) (unit 1)
     (in_bom yes) (on_board yes)
@@
     (pin "3")
     (pin "4")
+  )
+  (symbol (lib_id "Device:C") (at 156.21 137.16 0) (unit 1)
+    (in_bom yes) (on_board yes) (fields_autoplaced)
+    (property "Reference" "C14" (id 0) (at 160.02 135.8899 0)
+      (effects (font (size 1.27 1.27)) (justify left))
+    )
+    (property "Value" "0.1u" (id 1) (at 160.02 138.4299 0)
+      (effects (font (size 1.27 1.27)) (justify left))
+    )
+    (property "Footprint" "Capacitor_SMD:C_0603_1608Metric_Pad1.08x0.95mm_HandSolder" (id 2) (at 157.1752 140.97 0)
+      (effects (font (size 1.27 1.27)) hide)
+    )
+    (property "Datasheet" "~" (id 3) (at 156.21 137.16 0)
+      (effects (font (size 1.27 1.27)) hide)
+    )
+    (pin "1")
+    (pin "2")
   )
   (symbol (lib_id "power:GND") (at 201.93 67.31 0) (unit 1)
@@
     )
     (path "/4fd66cdc-862a-4ec3-a2f5-781967345f48"
-      (reference "#PWR?") (unit 1) (value "GND") (footprint "")
+      (reference "#PWR0103") (unit 1) (value "GND") (footprint "")
     )
     (path "/5e299d13-e854-4aa2-a425-a3ebf398ea1f"
@@
       (reference "C13") (unit 1) (value "12p") (footprint "Capacitor_SMD:C_0603_1608Metric_Pad1.08x0.95mm_HandSolder")
     )
+    (path "/d877682d-db4b-4e0e-842f-e25a34cf8eb8"
+      (reference "C14") (unit 1) (value "0.1u") (footprint "Capacitor_SMD:C_0603_1608Metric_Pad1.08x0.95mm_HandSolder")
+    )
+    (path "/cca679ce-7d8f-4c4e-96b3-4f48e0602970"
+      (reference "C15") (unit 1) (value "0.1u") (footprint "Capacitor_SMD:C_0603_1608Metric_Pad1.08x0.95mm_HandSolder")
+    )
     (path "/939411a5-54ee-4f8c-a422-9b8b80d3489a"
       (reference "D1") (unit 1) (value "LED") (footprint "LED_THT:LED_D3.0mm")
@@
     )
     (path "/2f215f15-3d52-4c91-93e6-3ea03a95622f"
-      (reference "U1") (unit 1) (value "RP2040") (footprint "IC57_RP2040")
+      (reference "U1") (unit 1) (value "RP2040") (footprint "Local:RP2040")
     )
     (path "/86f585ae-7fec-451b-9f4d-5178606c3d7d"
